Commit message: Working hydro branch

File: razbot_description/urdf/razbot.urdf.xacro (robot description, xacro)
@@ -17,5 +17,5 @@
   <xacro:property name="wheel_radius" value="0.040" />
   <!-- Calculated Properties -->
-  <xacro:property name="base_vertical_offset" value="${wheel_radius-wheel_vertical_offset}" />
+  <xacro:property name="base_vertical_offset" value="0.040" />
   <!-- <material> tags are used to describe the colour of robot components -->
   <material name="Blue">

File: razbot_description/urdf/wheel.urdf.xacro (robot description, xacro)
@@ -45,4 +45,5 @@
       <actuator name="${wheel_prefix}_wheel_motor">
         <mechanicalReduction>1</mechanicalReduction>
+        <hardwareInterface>VelocityJointInterface</hardwareInterface>
       </actuator>
       <joint name="${wheel_prefix}_wheel">
